File: BEEWATCH/GPS.kicad_sch (KiCad schematic)
At the start: 7 parts, among them U8 MPU-6050

Commit message: Save Kicad files
Parts:
- renumbered C24 to C17, C17 to C19, C16 to C20, R21 to R13, R22 to R14, U8 to U?
Changed lines of the file:
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@@
   (symbol (lib_id "Device:C_Small") (at 112.395 78.74 0) (unit 1)
     (in_bom yes) (on_board yes) (dnp no) (fields_autoplaced)
-    (property "Reference" "C24" (at 114.935 78.1113 0)
+    (property "Reference" "C17" (at 114.935 78.1113 0)
       (effects (font (size 1.27 1.27)) (justify left))
     )
@@
       (project "BEEWATCH"
         (path "/e9c5fb53-480b-4989-8495-a3341ee99514/45e7f89e-d204-4195-8987-9a9b7a51f032"
-          (reference "C24") (unit 1)
+          (reference "C17") (unit 1)
         )
       )
@@
   (symbol (lib_id "Device:C_Small") (at 178.435 113.665 0) (unit 1)
     (in_bom yes) (on_board yes) (dnp no) (fields_autoplaced)
-    (property "Reference" "C17" (at 181.61 113.0363 0)
+    (property "Reference" "C19" (at 181.61 113.0363 0)
       (effects (font (size 1.27 1.27)) (justify left))
     )
@@
       (project "BEEWATCH"
         (path "/e9c5fb53-480b-4989-8495-a3341ee99514/45e7f89e-d204-4195-8987-9a9b7a51f032"
-          (reference "C17") (unit 1)
+          (reference "C19") (unit 1)
         )
       )
@@
   (symbol (lib_id "Device:C_Small") (at 166.37 114.3 0) (unit 1)
     (in_bom yes) (on_board yes) (dnp no) (fields_autoplaced)
-    (property "Reference" "C16" (at 168.91 113.6713 0)
+    (property "Reference" "C20" (at 168.91 113.6713 0)
       (effects (font (size 1.27 1.27)) (justify left))
     )
@@
       (project "BEEWATCH"
         (path "/e9c5fb53-480b-4989-8495-a3341ee99514/45e7f89e-d204-4195-8987-9a9b7a51f032"
-          (reference "C16") (unit 1)
+          (reference "C20") (unit 1)
         )
       )
@@
   (symbol (lib_id "Device:R_Small") (at 120.65 109.22 90) (unit 1)
     (in_bom yes) (on_board yes) (dnp no)
-    (property "Reference" "R22" (at 120.65 111.76 90)
+    (property "Reference" "R14" (at 120.65 111.76 90)
       (effects (font (size 1.27 1.27)))
     )
@@
       (project "BEEWATCH"
         (path "/e9c5fb53-480b-4989-8495-a3341ee99514/45e7f89e-d204-4195-8987-9a9b7a51f032"
-          (reference "R22") (unit 1)
+          (reference "R14") (unit 1)
         )
       )
@@
   (symbol (lib_id "Sensor_Motion:MPU-6050") (at 142.24 101.6 0) (unit 1)
     (in_bom yes) (on_board yes) (dnp no)
-    (property "Reference" "U8" (at 129.54 85.725 0)
+    (property "Reference" "U?" (at 129.54 85.725 0)
       (effects (font (size 1.27 1.27)) (justify left))
     )
@@
       (project "BEEWATCH"
         (path "/e9c5fb53-480b-4989-8495-a3341ee99514"
-          (reference "U8") (unit 1)
-        )
-        (path "/e9c5fb53-480b-4989-8495-a3341ee99514/45e7f89e-d204-4195-8987-9a9b7a51f032"
-          (reference "U3") (unit 1)
+          (reference "U?") (unit 1)
+        )
+        (path "/e9c5fb53-480b-4989-8495-a3341ee99514/45e7f89e-d204-4195-8987-9a9b7a51f032"
+          (reference "U4") (unit 1)
         )
       )
@@
   (symbol (lib_id "Device:R_Small") (at 120.65 106.68 90) (unit 1)
     (in_bom yes) (on_board yes) (dnp no)
-    (property "Reference" "R21" (at 120.65 104.775 90)
+    (property "Reference" "R13" (at 120.65 104.775 90)
       (effects (font (size 1.27 1.27)))
     )
@@
       (project "BEEWATCH"
         (path "/e9c5fb53-480b-4989-8495-a3341ee99514/45e7f89e-d204-4195-8987-9a9b7a51f032"
-          (reference "R21") (unit 1)
-        )
-      )
+          (reference "R13") (unit 1)
+        )
+      )

Commit message: Insufficient GPIOs planning to add/C MUX or MCU
Changed lines of the file:
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@@
     (effects (font (size 1.27 1.27)) (justify left bottom))
   )
-  (hierarchical_label "MPU_SDA" (shape input) (at 123.19 93.98 180) (fields_autoplaced)
+  (hierarchical_label "MPU_SDA" (shape bidirectional) (at 123.19 93.98 180) (fields_autoplaced)
     (effects (font (size 1.27 1.27)) (justify right))
   )
@@
     (effects (font (size 1.27 1.27)) (justify right))
   )
-  (hierarchical_label "MPU_INT" (shape input) (at 164.465 93.98 0) (fields_autoplaced)
+  (hierarchical_label "MPU_INT" (shape output) (at 164.465 93.98 0) (fields_autoplaced)
     (effects (font (size 1.27 1.27)) (justify left))
   )
