File: Kicad/BEEWATCH MK3/Display.kicad_sch (KiCad schematic)
At the start: 6 parts, among them J3 Conn_02x06_Odd_Even, Q2 2N7002

Commit message: Rough layout placement
Parts:
- removed Q2: 2N7002, Package_TO_SOT_SMD:SOT-23, symbol Transistor_FET:2N7002
- added Q2: DMG6968U, Package_TO_SOT_SMD:SOT-23, symbol Transistor_FET:DMG2302U
Connections:
- net +3.3V: now also J3.4 (Pin_4); no longer J3.10 (Pin_10)
- net GND: now also J3.10 (Pin_10), J3.12 (Pin_12), Q2.2 (S); no longer J3.2 (Pin_2), J3.4 (Pin_4)
- net TFT_CS: now also J3.9 (Pin_9); no longer J3.5 (Pin_5)
- net TFT_D/C: now also J3.11 (Pin_11); no longer J3.7 (Pin_7)
- net TFT_LEDK: now also J3.3 (Pin_3), Q2.3 (D); no longer J3.11 (Pin_11)
- net TFT_RST: now also J3.2 (Pin_2); no longer J3.12 (Pin_12)
- net TFT_SCK: now also J3.7 (Pin_7); no longer J3.3 (Pin_3)
- net TFT_SDI: now also J3.5 (Pin_5); no longer J3.1 (Pin_1)
- net at R17.2, R18.1: now also Q2.1 (G)
- net TFT_LEDA: now reaches R19.1
- net TFT_LEDA: now also J3.1 (Pin_1); no longer J3.9 (Pin_9)
Other:
- moved on the sheet: C18, R19
