File: Kicad/BEEWATCH MK3/ESP32.kicad_sch (KiCad schematic)
At the start: 37 parts, among them Q1 2N7002, SW1 TK-074-4, SW2 TK-074-4, U1 ESP32-S3, Y1 40MHz

Commit message: Rough layout placement
Parts:
- removed BZ1: BUZZER, Project:CL9032A-CLDZ-SMD Passive Buzzer, symbol OLED_WATCH-rescue:BUZZER-OLED_MOSFETs
- removed Q1: 2N7002, Package_TO_SOT_SMD:SOT-23, symbol Transistor_FET:2N7002
- added BZ2: Buzzer, Project:CL9032A-CLDZ-SMD Passive Buzzer, symbol Device:Buzzer
- added Q1: DMG6968U, Package_TO_SOT_SMD:SOT-23, symbol Transistor_FET:DMG2302U
- added R23: 5M, Resistor_SMD:R_0402_1005Metric, symbol Device:R
- C? (x4): footprint Capacitor_SMD:C_0603_1608Metric -> Capacitor_SMD:C_0201_0603Metric
- D1: footprint (none) -> LED_SMD:LED_WS2812B_PLCC4_5.0x5.0mm_P3.2mm
Connections:
- net +VBAT: now also BZ2.1 (+)
- net CHG_ST: now also U1.39 (GPIO34)
- net GND: now also Q1.2 (S)
- net LED1: now also U1.38 (GPIO33); no longer U1.27 (GPIO21)
- net XTAL_N: now also C?.1, Y1.1, R23.1; no longer C?.1, Y1.4
- net XTAL_P: now also C?.1, Y1.4, R23.2; no longer C?.1, Y1.1
- net BUZZER_EN: now reaches U1.40 (GPIO35)
- net BAT_ST_EN: now reaches U1.41 (GPIO36)
- net at R10.2, R9.2: now also Q1.1 (G)
- new net: BZ2.2 (-), Q1.3 (D)
- new net LCD_LED: U1.27 (GPIO21)
- no-connect marks 27 -> 23
Other:
- moved on the sheet: C?, R4, Y1, Y?
