File: Kicad/BEEWATCH MK3/RYS8830.kicad_sch (KiCad schematic)
At the start: 30 parts, among them Q4 BSS138, Q5 BSS138, Q6 BSS138, Q7 BSS138, U6 LTC3549EDCB#TRMPBF, U7 RYS8830

Commit message: Rough layout placement
Parts:
- U6: footprint Project:SON50P300X200X80-7N-D -> SON50P300X200X80-7N-D
Changed lines of the file:
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@@
 	(label "TXD"
 		(at 182.88 72.39 0)
-		(fields_autoplaced yes)
 		(effects
 			(font
@@
 	(label "RXD"
 		(at 182.88 68.58 0)
-		(fields_autoplaced yes)
 		(effects
 			(font
@@
 	(label "GNSS_+1.8V"
 		(at 59.69 68.58 0)
-		(fields_autoplaced yes)
 		(effects
 			(font
@@
 	(label "PPS"
 		(at 182.88 76.2 0)
-		(fields_autoplaced yes)
 		(effects
 			(font
@@
 		(shape input)
 		(at 54.61 48.26 180)
-		(fields_autoplaced yes)
 		(effects
 			(font
@@
 		(shape input)
 		(at 247.65 59.69 0)
-		(fields_autoplaced yes)
 		(effects
 			(font
@@
 		(shape output)
 		(at 247.65 83.82 0)
-		(fields_autoplaced yes)
 		(effects
 			(font
@@
 		(shape output)
 		(at 248.92 119.38 0)
-		(fields_autoplaced yes)
 		(effects
 			(font
@@
 		(shape input)
 		(at 248.92 135.89 0)
-		(fields_autoplaced yes)
 		(effects
 			(font
@@
 			)
 		)
-		(property "Description" ""
+		(property "Description" "Resistor"
 			(at 208.28 53.34 0)
 			(effects
@@
 			)
 		)
-		(property "Description" ""
+		(property "Description" "50V Vds, 0.22A Id, N-Channel MOSFET, SOT-23"
 			(at 219.71 57.15 0)
 			(effects
@@
 			)
 		)
-		(property "Description" ""
+		(property "Description" "Resistor"
 			(at 228.6 90.17 0)
 			(effects
@@
 			)
 		)
-		(property "Description" ""
+		(property "Description" "Power symbol creates a global label with name \"+3.3V\""
 			(at 85.09 31.75 0)
 			(effects
@@
 			)
 		)
-		(property "Description" ""
+		(property "Description" "Power symbol creates a global label with name \"+3.3V\""
 			(at 209.55 152.4 0)
 			(effects
@@
 			)
 		)
-		(property "Description" ""
+		(property "Description" "50V Vds, 0.22A Id, N-Channel MOSFET, SOT-23"
 			(at 73.66 45.72 0)
 			(effects
@@
 			)
 		)
-		(property "Description" ""
+		(property "Description" "Power symbol creates a global label with name \"+5V\""
 			(at 228.6 100.33 0)
 			(effects
@@
 			)
 		)
-		(property "Description" ""
+		(property "Description" "Resistor"
 			(at 208.28 90.17 0)
 			(effects
@@
 			)
 		)
-		(property "Description" ""
+		(property "Description" "Power symbol creates a global label with name \"+3.3V\""
 			(at 208.28 43.18 0)
 			(effects
@@
 			)
 		)
-		(property "Description" ""
+		(property "Description" "Power symbol creates a global label with name \"+3.3V\""
 			(at 163.83 102.87 0)
 			(effects
@@
 			)
 		)
-		(property "Description" ""
+		(property "Description" "Schottky diode"
 			(at 219.71 119.38 0)
 			(effects
@@
 			)
 		)
-		(property "Description" ""
+		(property "Description" "Resistor"
 			(at 64.77 41.91 0)
 			(effects
@@
 			)
 		)
-		(property "Description" ""
+		(property "Description" "Resistor"
 			(at 30.48 64.77 0)
 			(effects
@@
 			)
 		)
-		(property "Description" ""
+		(property "Description" "Power symbol creates a global label with name \"+5V\""
 			(at 64.77 31.75 0)
 			(effects
@@
 			)
 		)
-		(property "Description" ""
+		(property "Description" "Power symbol creates a global label with name \"+5V\""
 			(at 229.87 152.4 0)
 			(effects
@@
 			)
 		)
-		(property "Description" ""
+		(property "Description" "50V Vds, 0.22A Id, N-Channel MOSFET, SOT-23"
 			(at 220.98 138.43 0)
 			(effects
@@
 			)
 		)
-		(property "Description" ""
+		(property "Description" "Resistor"
 			(at 237.49 113.03 0)
 			(effects
@@
 			)
 		)
-		(property "Footprint" "Project:SON50P300X200X80-7N-D"
+		(property "Footprint" "SON50P300X200X80-7N-D"
 			(at 78.74 177.47 0)
 			(effects
@@
 			)
 		)
-		(property "Description" ""
+		(property "Description" "Resistor"
 			(at 228.6 53.34 0)
 			(effects
@@
 			)
 		)
-		(property "Description" ""
+		(property "Description" "Power symbol creates a global label with name \"+5V\""
 			(at 228.6 43.18 0)
 			(effects
@@
 			)
 		)
-		(property "Description" ""
+		(property "Description" "Power symbol creates a global label with name \"+3.3V\""
 			(at 30.48 60.96 0)
 			(effects
@@
 			)
 		)
-		(property "Description" ""
+		(property "Description" "Power symbol creates a global label with name \"+5V\""
 			(at 237.49 106.68 0)
 			(effects
@@
 			)
 		)
-		(property "Description" ""
+		(property "Description" "Power symbol creates a global label with name \"+3.3V\""
 			(at 208.28 100.33 0)
 			(effects
@@
 			)
 		)
-		(property "Description" ""
+		(property "Description" "Resistor"
 			(at 209.55 142.24 0)
 			(effects
@@
 			)
 		)
-		(property "Description" ""
+		(property "Description" "Resistor"
 			(at 85.09 41.91 0)
 			(effects
@@
 			)
 		)
-		(property "Description" ""
+		(property "Description" "50V Vds, 0.22A Id, N-Channel MOSFET, SOT-23"
 			(at 219.71 86.36 0)
 			(effects
@@
 			)
 		)
-		(property "Description" ""
+		(property "Description" "Resistor"
 			(at 229.87 142.24 0)
 			(effects
