File: Kicad/BEEWATCH MK2/BEEWATCH MK2.kicad_pcb (KiCad board)
At the start: 4 copper layers, 40.3 x 39.7 mm, 119 parts, among them J1 USB_C_Receptacle_USB2.0_16P, J3 Conn_02x06_Odd_Even, Q1 DMG6968U, Q2 DMG6968U, Q3 DMP1045U-7, Q4 DMG6968U, Q5 BSS138, Q6 BSS138, Q7 BSS138, Q8 DMP1045U-7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

Commit message: Deep optmizing the Layout
Parts:
- removed the Q3 at (141.0, 117.7)
- moved R45 45.4 mm to (96.8, 94.2), turned to 90 degrees
- moved R44 45.0 mm to (96.8, 96.7), turned to 90 degrees
- moved R46 43.8 mm to (97.5, 98.6), turned to 0 degrees
- moved C30 41.7 mm to (115.3, 95.3), turned to -90 degrees
- moved Q9 40.6 mm to (99.2, 95.5), turned to 90 degrees
- moved R47 38.6 mm to (100.3, 98.6), turned to 0 degrees
- moved BT1 37.9 mm to (164.4, 75.2)
- moved U8 36.5 mm to (118.1, 93.9), turned to 90 degrees
- moved C31 35.8 mm to (117.8, 97.0), turned to 180 degrees
- moved R25 30.1 mm to (132.6, 98.5), turned to 135 degrees
- moved R26 28.3 mm to (138.9, 89.1), turned to -135 degrees
- moved R27 27.9 mm to (139.7, 90.7), turned to -45 degrees
- moved C28 27.4 mm to (138.3, 91.3), turned to 135 degrees
- moved R40 27.2 mm to (178.4, 123.1)
- moved R36 26.9 mm to (128.3, 119.9)
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Routing:
- net VBUS: track 25.5 -> 0.00 mm
- net /Battery&BMS/VBAT: track 19.3 -> 0.00 mm
- net /Battery&BMS/+VBAT_IN: track 12.6 -> 0.00 mm
- net GND: track 10.6 -> 0.00 mm, vias 3 -> 0
- net /ESP32/GPS_TXD: track 7.32 -> 0.00 mm, vias 1 -> 0
- net +3.3V: track 5.57 -> 0.00 mm, vias 2 -> 0
- net /ACCELEROMETER/MPU_SDA: track 4.46 -> 0.00 mm
- net /ESP32/XTAL_32K_N: track 4.38 -> 0.00 mm
- net Net-(J1-CC1): track 4.02 -> 0.00 mm
- net /ESP32/USB_D+: track 3.97 -> 0.00 mm
- net /ESP32/USB_D-: track 3.94 -> 0.00 mm
- net VDD3P3_RTC: track 3.53 -> 0.00 mm
- net /ESP32/XTAL_32K_P: track 3.34 -> 0.00 mm
- net Net-(U4-STAT): track 3.17 -> 0.00 mm
- net /ESP32/GPS_RXD: track 3.07 -> 0.00 mm, vias 1 -> 0
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