File: Kicad/BEEWATCH MK2 PANALIZED/BEEWATCH MK2.kicad_pcb (KiCad board)
At the start: 4 copper layers, 100 x 40.6 mm, 130 parts, among them J1 USB_C_Receptacle_USB2.0_16P, J3 Conn_02x06_Odd_Even, J4 Conn_02x06_Odd_Even, Q1 DMG6968U, Q2 DMG6968U, Q3 DMP1045U-7, Q4 DMG6968U, Q5 BSS138, Q6 BSS138, Q7 BSS138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

Commit message: PCB Updated
Parts:
- removed the G*** at (183.6, 105.2)
- removed the G*** at (183.6, 105.1)
- added ?: , , F.Cu at (158.6, 88.2)
- added ?: , , F.Cu at (162.5, 119.0)
- added ?: , , F.Cu at (141.5, 88.3)
- added ?: , , B.Cu at (116.0, 88.3)
- added ?: , , B.Cu at (98.9, 88.2)
- added ?: , , B.Cu at (95.0, 119.0)
- moved J4 0.13 mm to (107.5, 121.3)
Routing:
- net /ESP32/D+: track 11.5 -> 13.0 mm, vias 1 -> 3
- net /ESP32/D-: track 14.6 -> 13.1 mm, vias 3 -> 1
- net /RYS8830/GNSS_+1.8V: track 100.5 -> 101.4 mm
- net /ACCELEROMETER/MPU_SDA: track 18.6 -> 18.0 mm
Other:
- board size 100 x 40.6 mm -> 82.8 x 40.3 mm
